Commit message: update new_gimbal_controller

File: rotors_description/urdf/multirotor_base.xacro (robot description, xacro)
@@ -35,4 +35,31 @@
     params="robot_namespace mass body_width body_height use_mesh_file mesh_file *inertia">
     <link name="${robot_namespace}/base_link"></link>
+    <!-- Included gimbal base link -->
+    <link name="${robot_namespace}/gimbal_base_link">
+      <inertial>
+        <origin xyz="0 0 -0.025" rpy="0 0 0" />
+        <mass value="0.1" />
+        <inertia ixx="5e-2" ixy="0.0" ixz="0.0" iyy="5e-2" iyz="0.0" izz="5e-2" />
+      </inertial>
+      <visual>
+        <origin xyz="0 0 -0.025" rpy="0 0 0"/>
+        <geometry>
+          <cylinder radius="0.025" length="0.01"/>
+        </geometry>
+        <material name="white"/>
+      </visual>
+    </link>
+    <joint name="${robot_namespace}/gimbal_pitch_joint" type="continuous">
+      <parent link="${robot_namespace}/base_link" />
+      <child link="${robot_namespace}/gimbal_base_link" />
+      <origin xyz="0 0 0" rpy="0 0 0" />
+      <axis xyz="0 1.570796 0" />
+    </joint>
+    <gazebo>
+      <plugin name="gimbal_controller_plugin" filename="librotors_gazebo_gimbal_plugin.so">
+        <linkBaseName>${robot_namespace}/base_link</linkBaseName>
+        <linkPitchName>${robot_namespace}/gimbal_base_link</linkPitchName>
+      </plugin>
+    </gazebo>
     <joint name="${robot_namespace}/base_joint" type="fixed">
       <origin xyz="0 0 0" rpy="0 0 0" />

File: rotors_description/urdf/vi_sensor_base.xacro (robot description, xacro)
@@ -18,7 +18,7 @@
     </visual>
     <inertial>
-      <mass value="100" />
+      <mass value="0.001" />
       <origin xyz="0 0 0" rpy="0 0 0" />
-      <inertia ixx="1" ixy="0" ixz="0" iyy="1" iyz="0" izz="1" />
+      <inertia ixx="1e-6" ixy="0" ixz="0" iyy="1e-6" iyz="0" izz="1e-6" />
     </inertial>
   </link>
